File: open/relay_module_24v/relay_module_24v.kicad_pcb (KiCad board)
At the start: 2 copper layers, 30.5 x 61 mm, 10 parts, among them J1 Conn_01x02_Pin, J2 Conn_01x03_Pin, K1 Relay_SPDT

Commit message: v1.0.0
Changed lines of the file:
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@@
+	)
+	(segment
+		(start 142.961 132.834)
+		(end 144.061 133.934)
+		(width 3.5)
+		(layer "B.Cu")
+		(net 2)
 	)
 	(segment
 		(start 142.961 120.172)
 		(end 142.961 132.834)
-		(width 2)
+		(width 3.5)
 		(layer "B.Cu")
 		(net 2)
 	)
 	(segment
-		(start 142.961 132.834)
-		(end 144.061 133.934)
-		(width 2)
+		(start 148.961 133.754)
+		(end 149.141 133.934)
+		(width 3.5)
 		(layer "B.Cu")
-		(net 2)
+		(net 3)
 	)
 	(segment
 		(start 148.961 105.972)
 		(end 148.961 133.754)
-		(width 2)
+		(width 3.5)
 		(layer "B.Cu")
 		(net 3)
 	)
 	(segment
-		(start 148.961 133.754)
-		(end 149.141 133.934)
-		(width 2)
+		(start 154.961 133.194)
+		(end 154.221 133.934)
+		(width 3.5)
 		(layer "B.Cu")
-		(net 3)
+		(net 4)
 	)
 	(segment
 		(start 154.961 120.172)
 		(end 154.961 133.194)
-		(width 2)
+		(width 3.5)
 		(layer "B.Cu")
 		(net 4)
-	)
-	(segment
-		(start 154.961 133.194)
-		(end 154.221 133.934)
-		(width 2)
-		(layer "B.Cu")
-		(net 4)
