File: open/relay_module_12v_optocoupler/relay_module_12v_optocoupler.kicad_sch (KiCad schematic)
At the start: 11 parts, among them J1 Conn_01x02_Pin, J2 Conn_01x03_Pin, K1 Relay_SPDT, Q1 BC337, U1 PC817

Commit message: v1.0.0
Connections:
- net GND: now also J1.2 (Pin_2); no longer D2.1 (K), J1.3 (Pin_3)
- net at R2.1: now also J1.3 (Pin_3); no longer J1.1 (Pin_1)
- net at D1.1 (K), K1.1, R1.1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: now also J1.1 (Pin_1); no longer J1.2 (Pin_2)
- net at D1.2 (A), K1.2, Q1.1 (C): now also D2.1 (K)
Other:
- moved on the sheet: D1, D2, J1, J2, K1, Q1, R1, R2, R3, R4, U1
