File: carrier_board_arduino_current_driver/carrier_board_arduino_current_driver.kicad_pcb (KiCad board)
At the start: 2 copper layers, 61.4 x 49.7 mm, 17 parts, among them J1 Conn_01x03_Pin, J3 Barrel_Jack, Q1 TIP41, Q2 TIP42, U1 L7805

Commit message: v1.0.0
Parts:
- removed REF** (x4): MH, MountingHole:MountingHole_3.2mm_M3
- added D1: 1N4007, Diode_THT:D_DO-41_SOD81_P10.16mm_Horizontal, F.Cu at (207.6, 57.0)
- added D2: LED, LED_THT:LED_D3.0mm, F.Cu at (193.7, 51.9)
- added D3: 1N4007, Diode_THT:D_DO-41_SOD81_P10.16mm_Horizontal, F.Cu at (188.0, 55.2)
- added D4: 1N4007, Diode_THT:D_DO-41_SOD81_P10.16mm_Horizontal, F.Cu at (188.0, 76.3)
- added J2: Conn_01x03_Pin, TerminalBlock_Phoenix:TerminalBlock_Phoenix_MKDS-1,5-3-5.08_1x03_P5.08mm_Horizontal, F.Cu at (195.0, 89.5)
- added JP1: Jumper_3_Open, Connector_PinHeader_2.54mm:PinHeader_1x03_P2.54mm_Vertical, F.Cu at (153.5, 74.5)
- added K1: Relay_SPDT, Relay_THT:Relay_SPDT_Omron-G5LE-1, F.Cu at (200.1, 62.9)
- added Q3: BC337, Package_TO_SOT_THT:TO-92_Inline, F.Cu at (193.7, 57.1)
- added R10: R, Resistor_THT:R_Axial_DIN0207_L6.3mm_D2.5mm_P7.62mm_Horizontal, F.Cu at (178.4, 38.2)
- added R11: 1k, Resistor_THT:R_Axial_DIN0207_L6.3mm_D2.5mm_P7.62mm_Horizontal, F.Cu at (154.5, 92.5)
- added R5: R, Resistor_THT:R_Axial_DIN0207_L6.3mm_D2.5mm_P7.62mm_Horizontal, F.Cu at (191.1, 39.9)
- added R6: R, Resistor_THT:R_Axial_DIN0207_L6.3mm_D2.5mm_P7.62mm_Horizontal, F.Cu at (198.8, 43.7)
- added R7: R, Resistor_THT:R_Axial_DIN0207_L6.3mm_D2.5mm_P7.62mm_Horizontal, F.Cu at (198.8, 47.5)
- added R8: R, Resistor_THT:R_Axial_DIN0207_L6.3mm_D2.5mm_P7.62mm_Horizontal, F.Cu at (207.6, 51.9)
- added R9: R, Resistor_THT:R_Axial_DIN0207_L6.3mm_D2.5mm_P7.62mm_Horizontal, F.Cu at (182.2, 38.2)
- added U2: PC817, Package_DIP:DIP-4_W7.62mm, F.Cu at (207.0, 40.5)
- added U3: LM358, Package_DIP:DIP-8_W7.62mm, F.Cu at (165.7, 84.8)
- Q1: value TIP41 -> TIP4x/ TIP12x
- Q2: value TIP42 -> TIP4x/ TIP12x
- R3: value R -> 68k
- R4: value R -> 39k
- moved R1 74.1 mm to (181.6, 66.7), turned to 90 degrees
- moved R2 72.1 mm to (177.8, 66.7), turned to 90 degrees
- moved A1 70.7 mm to (173.4, 79.4)
- moved C2 59.3 mm to (154.0, 62.3), turned to -90 degrees
- moved Q1 57.8 mm to (184.8, 49.2), turned to 180 degrees
- moved Q2 55.1 mm to (185.2, 70.6), turned to 180 degrees
- moved J1 53.6 mm to (178.4, 89.5), turned to 0 degrees
- moved C1 46.3 mm to (149.5, 57.0), turned to 0 degrees
- moved U1 43.1 mm to (150.4, 69.0), turned to 90 degrees
- moved J3 41.9 mm to (150.8, 51.1)
- moved R3 38.4 mm to (147.5, 84.9), turned to -90 degrees
- moved R4 35.1 mm to (151.0, 92.5), turned to 90 degrees
- moved RV1 23.4 mm to (148.5, 80.5), turned to 180 degrees
Connections:
- A1 pad 9: unconnected-(A1-D6-Pad9) -> D6
- C1 pad 1: Net-(Q2-E) -> Net-(JP1-B)
- J3 pad 1: Net-(Q2-E) -> Net-(JP1-B)
- Q2 pad 3: Net-(Q2-E) -> Net-(D1-K)
- R3 pad 1: Net-(A1-A0) -> Net-(R11-Pad2)
- R4 pad 2: Net-(A1-A0) -> Net-(R11-Pad2)
- U1 pad 1: Net-(Q2-E) -> Net-(JP1-B)
Routing:
- net GND: track 200.6 -> 0.00 mm
- net Net-(Q2-E): track 50.0 -> 0.00 mm
- net Net-(A1-+5V): track 32.1 -> 0.00 mm
- net Net-(A1-A0): track 67.3 -> 35.5 mm
- net Net-(Q2-B): track 16.9 -> 0.00 mm
- net A0: track 15.8 -> 0.00 mm
- net Net-(D3-A): track 31.3 -> 17.1 mm
- net Net-(Q1-B): track 22.8 -> 8.82 mm
- net Net-(R5-Pad2): track 0.00 -> 10.1 mm
- net Net-(D1-K): track 0.00 -> 9.15 mm
- net Net-(R4-Pad1): track 8.83 -> 0.00 mm
- net Net-(D1-A): track 0.00 -> 8.32 mm
- net Net-(R6-Pad1): track 0.00 -> 7.56 mm
- net Net-(R11-Pad2): track 0.00 -> 7.00 mm
- net Net-(JP1-B): track 0.00 -> 6.46 mm
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Other:
- board size 61.4 x 49.7 mm -> 68.5 x 61.8 mm

Commit message: v1.0.0
Parts:
- removed D1: 1N4007, Diode_THT:D_DO-41_SOD81_P10.16mm_Horizontal
- removed D2: LED, LED_THT:LED_D3.0mm
- removed J2: Conn_01x03_Pin, TerminalBlock_Phoenix:TerminalBlock_Phoenix_MKDS-1,5-3-5.08_1x03_P5.08mm_Horizontal
- removed K1: Relay_SPDT, Relay_THT:Relay_SPDT_Omron-G5LE-1
- removed Q3: BC337, Package_TO_SOT_THT:TO-92_Inline
- added C3: 10uF 16V, Capacitor_SMD:CP_Elec_6.3x5.4, F.Cu at (151.1, 52.5)
- added R12: 1k, Resistor_SMD:R_0805_2012Metric, F.Cu at (183.2, 75.6)
- added REF**: MountingHole_2.2mm_M2, MountingHole:MountingHole_2.2mm_M2, F.Cu at (192.4, 80.0)
- added REF**: MountingHole_2.2mm_M2, MountingHole:MountingHole_2.2mm_M2, F.Cu at (192.4, 37.5)
- added REF**: MountingHole_2.2mm_M2, MountingHole:MountingHole_2.2mm_M2, F.Cu at (139.7, 80.0)
- added REF**: MountingHole_2.2mm_M2, MountingHole:MountingHole_2.2mm_M2, F.Cu at (139.7, 37.5)
- added U4: PC817, Package_SO:SO-4_4.4x3.6mm_P2.54mm, F.Cu at (178.5, 39.9)
- C1: value C_Polarized -> 100uF 16V; footprint Capacitor_THT:CP_Radial_D6.3mm_P2.50mm -> Capacitor_SMD:CP_Elec_6.3x5.4
- C2: value C -> 100nF; footprint Capacitor_THT:C_Disc_D5.0mm_W2.5mm_P5.00mm -> Capacitor_SMD:C_0603_1608Metric
- D3, D4: footprint Diode_THT:D_DO-41_SOD81_P10.16mm_Horizontal -> Diode_SMD:D_SOD-123
- J1: footprint TerminalBlock_Phoenix:TerminalBlock_Phoenix_MKDS-1,5-3-5.08_1x03_P5.08mm_Horizontal -> Connector_PinHeader_2.54mm:PinHeader_1x04_P2.54mm_Vertical
- R1, R10, R11, R2, R3, R4, R5, R6, R9: footprint Resistor_THT:R_Axial_DIN0207_L6.3mm_D2.5mm_P7.62mm_Horizontal -> Resistor_SMD:R_0805_2012Metric
- R7: value R -> 68k; footprint Resistor_THT:R_Axial_DIN0207_L6.3mm_D2.5mm_P7.62mm_Horizontal -> Resistor_SMD:R_0805_2012Metric
- R8: value R -> 39k; footprint Resistor_THT:R_Axial_DIN0207_L6.3mm_D2.5mm_P7.62mm_Horizontal -> Resistor_SMD:R_0805_2012Metric
- U1: footprint Package_TO_SOT_THT:TO-220-3_Vertical -> Package_TO_SOT_SMD:TO-252-2
- U2: footprint Package_DIP:DIP-4_W7.62mm -> Package_SO:SO-4_4.4x3.6mm_P2.54mm
- U3: footprint Package_DIP:DIP-8_W7.62mm -> Package_SO:SOIC-8_3.9x4.9mm_P1.27mm
- moved R4 42.8 mm to (183.2, 64.3)
- moved RV1 41.1 mm to (187.5, 67.5), turned to 90 degrees
- moved R3 39.1 mm to (180.8, 64.3)
- moved R8 37.9 mm to (178.0, 75.6), turned to 90 degrees
- moved R11 36.8 mm to (178.2, 64.3)
- moved R7 33.4 mm to (180.7, 75.6), turned to -90 degrees
- moved D4 33.1 mm to (183.0, 43.6), turned to -90 degrees
- moved JP1 31.9 mm to (154.2, 42.6), turned to 180 degrees
- moved U2 30.8 mm to (178.7, 52.5), turned to 90 degrees
- moved R1 30.3 mm to (182.9, 36.4), turned to 0 degrees
- moved R5 22.5 mm to (178.7, 58.6)
- moved U3 20.9 mm to (180.6, 70.1), turned to 0 degrees
- moved R6 20.3 mm to (178.6, 46.0), turned to 0 degrees
- moved Q2 19.9 mm to (186.5, 50.8), turned to -90 degrees
- moved R2 18.3 mm to (182.9, 49.1), turned to 0 degrees
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Connections:
- A1 pad 19: Net-(A1-A0) -> unconnected-(A1-A0-Pad19)
- A1 pad 25: unconnected-(A1-A6-Pad25) -> A6
- A1 pad 26: unconnected-(A1-A7-Pad26) -> A7
- A1 pad 29: unconnected-(A1-GND-Pad29) -> GND
- A1 pad 9: D6 -> unconnected-(A1-D6-Pad9)
- D3 pad 1: Net-(D1-K) -> Net-(D3-K)
- J1 pad 2: GND -> S1
- J1 pad 3: A0 -> S2
- JP1 pad 2: Net-(D1-K) -> Net-(D3-K)
- Q2 pad 3: Net-(D1-K) -> Net-(D3-K)
- R1 pad 1: Net-(A1-D5) -> D5
- R2 pad 1: Net-(A1-D3) -> D3
- R3 pad 2: A0 -> S1
- R5 pad 1: D6 -> Net-(A1-D3)
- R6 pad 1: Net-(R6-Pad1) -> Net-(A1-D5)
- R6 pad 2: Net-(Q3-B) -> Net-(R6-Pad2)
- R7 pad 1: GND -> Net-(R12-Pad2)
- R7 pad 2: Net-(Q3-B) -> S2
- R8 pad 1: Net-(D1-K) -> GND
- R8 pad 2: Net-(D2-A) -> Net-(R12-Pad2)
- RV1 pad 2: GND -> Net-(R4-Pad1)
- U2 pad 3: Net-(R6-Pad1) -> D3
- U2 pad 4: Net-(D1-K) -> Net-(D3-K)
- U3 pad 1: Net-(A1-A0) -> A6
- U3 pad 2: Net-(A1-A0) -> A6
- U3 pad 4: (no net) -> GND
- U3 pad 5: (no net) -> Net-(U3B-+)
- U3 pad 6: (no net) -> A7
- U3 pad 7: (no net) -> A7
- U3 pad 8: (no net) -> Net-(D3-K)
Routing:
- net Net-(D3-K): track 0.00 -> 77.8 mm, vias 0 -> 4
- net Net-(A1-+5V): track 0.00 -> 67.7 mm
- net A7: track 0.00 -> 45.2 mm
- net A6: track 0.00 -> 43.4 mm
- net Net-(D3-A): track 17.1 -> 53.7 mm
- net Net-(A1-A0): track 35.5 -> 0.00 mm
- net Net-(JP1-B): track 6.46 -> 30.1 mm
- net S1: track 0.00 -> 18.2 mm
- net Net-(D1-K): track 9.15 -> 0.00 mm
- net Net-(U3A-+): track 0.00 -> 8.35 mm
- net Net-(D1-A): track 8.32 -> 0.00 mm
- net Net-(R4-Pad1): track 0.00 -> 7.75 mm
- net Net-(R6-Pad1): track 7.56 -> 0.00 mm
- net Net-(R5-Pad2): track 10.1 -> 3.81 mm
- net Net-(R12-Pad2): track 0.00 -> 6.10 mm
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- added copper zone on F.Cu, net GND
Other:
- board size 68.5 x 61.8 mm -> 57.5 x 47.5 mm
- board text added: "ANCB current drive v1.0"
