File: carrier_board_arduino_relay/carrier_board_arduino_current_driver.kicad_sch (KiCad schematic)
At the start: 28 parts, among them J1 Conn_01x03_Pin, J3 Barrel_Jack, Q1 TIP4x/ TIP12x, Q2 TIP4x/ TIP12x, U1 L7805, U2 PC817, U3 LM358, U4 PC817

Commit message: v1.0.0
Parts:
- removed C3: 10uF 16V, Capacitor_SMD:CP_Elec_6.3x5.4, symbol Device:C_Polarized
- removed R12: 1k, Resistor_SMD:R_0805_2012Metric, symbol Device:R
- removed unit 2 of U3
- removed unit 3 of U3
- removed U4: PC817, Package_SO:SO-4_4.4x3.6mm_P2.54mm, symbol Isolator:PC817
- added D1: 1N4007, Diode_SMD:D_SOD-123, symbol Diode:1N4007
- added D2: LED, LED_SMD:LED_0805_2012Metric, symbol Device:LED
- added J2: Conn_01x03_Pin, TerminalBlock_Phoenix:TerminalBlock_Phoenix_MKDS-1,5-3-5.08_1x03_P5.08mm_Horizontal, symbol Connector:Conn_01x03_Pin
- added K1: Relay_SPDT, Relay_THT:Relay_SPDT_Omron-G5LE-1, symbol Relay:Relay_SPDT
- added Q3: BC817, Package_TO_SOT_SMD:SOT-23, symbol Transistor_BJT:BC817
- C1: value 100uF 16V -> C_Polarized; footprint Capacitor_SMD:CP_Elec_6.3x5.4 -> Capacitor_THT:CP_Radial_D6.3mm_P2.50mm
- C2: value 100nF -> C; footprint Capacitor_SMD:C_0603_1608Metric -> Capacitor_THT:C_Disc_D5.0mm_W2.5mm_P5.00mm
- J1: footprint Connector_PinHeader_2.54mm:PinHeader_1x04_P2.54mm_Vertical -> Connector_PinHeader_2.54mm:PinHeader_1x03_P2.54mm_Vertical; symbol Connector:Conn_01x04_Pin -> Connector:Conn_01x03_Pin
- R7: value 68k -> R
- R8: value 39k -> R
- U2: footprint Package_SO:SO-4_4.4x3.6mm_P2.54mm -> Package_DIP:DIP-4_W7.62mm
Connections:
- net D5 is gone; now on an unnamed net: R1.1
- net GND: now also J1.2 (Pin_2), R7.1, RV1.2, Q3.2 (E); no longer A1.29 (GND), J1.4 (Pin_4), R8.1
- net at D3.1 (K), JP1.2 (C), Q2.3 (E)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: now also R8.1, D1.1 (K), K1.1
- net at A1.19 (A0): now also U3.1, U3.2 (-)
- net at A1.6 (D3): now also R2.1; no longer R5.1
- net at A1.8 (D5): no longer R6.1
- net D6: now reaches A1.9 (D6)
- net D6: now also R5.1
- net at R4.1, RV1.1: no longer RV1.2
- net at R6.2: now also R7.2, Q3.1 (B)
- net at R8.2: now also D2.2 (A); no longer R7.1
- removed net A6: A1.25 (A6), U3.1, U3.2 (-)
- net A7: no longer names the net of A1.26 (A7)
- net D3: no longer names the net of U2.3
- net D3: now also R6.1; no longer R2.1
- net S1 renamed A0
- net A0: now also J1.3 (Pin_3); no longer J1.2 (Pin_2)
- removed net S2: J1.3 (Pin_3), R7.2
- new net: D1.2 (A), D2.1 (K), K1.2, Q3.3 (C)
- new net C_1: J2.2 (Pin_2), K1.3
- new net NC_1: J2.3 (Pin_3), K1.4
- new net NO_1: J2.1 (Pin_1), K1.5
Other:
- moved on the sheet: C2, D3, D4, Q1, Q2, R1, R10, R11, R2, R3, R4, R5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
