File: arduino_nano_low_side_cc_driver/arduino_nano_low_side_cc_driver.kicad_sch (KiCad schematic)
At the start: 31 parts, among them J1 Conn_01x06_Pin, J2 Conn_01x02_Pin, J3 Barrel_Jack, J4 Conn_01x02_Pin, Q1 IRF540N, Q2 IRF540N, U1 L7805, U2 PC817, U3 LM358, U4 PC817

Commit message: v1.0.0
Connections:
- net L1b: now also D2.1 (K), J1.1 (Pin_1), Q2.2 (D); no longer D1.1 (K), J1.5 (Pin_5), Q1.2 (D)
- net L2b: now also D1.1 (K), J1.5 (Pin_5), Q1.2 (D); no longer D2.1 (K), J1.1 (Pin_1), Q2.2 (D)
- net at R14.2, R16.2: now also Q1.1 (G); no longer Q2.1 (G)
- net at R1.2, R9.2: now also Q2.1 (G); no longer Q1.1 (G)
Other:
- moved on the sheet: D1, D2, Q1, Q2
Changed lines of the file:
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@@
 		)
 	)
-	(global_label "L1b"
+	(global_label "L2b"
 		(shape bidirectional)
 		(at 255.27 59.69 180)
@@
 		)
 	)
-	(global_label "L2a"
+	(global_label "L1a"
 		(shape bidirectional)
 		(at 255.27 67.31 180)
@@
 		)
 	)
-	(global_label "L1a"
+	(global_label "L2a"
 		(shape bidirectional)
 		(at 255.27 57.15 180)
@@
 		)
 	)
-	(global_label "L2b"
+	(global_label "L1b"
 		(shape bidirectional)
 		(at 255.27 69.85 180)
@@
 	(symbol
 		(lib_id "Diode:B120-E3")
-		(at 229.87 60.96 270)
+		(at 168.91 60.96 270)
 		(unit 1)
 		(exclude_from_sim no)
@@
 		(fields_autoplaced yes)
 		(property "Reference" "D2"
-			(at 232.41 60.6424 90)
+			(at 171.45 60.6424 90)
 			(effects
 				(font
@@
 		)
 		(property "Value" "B120-E3"
-			(at 232.41 61.9124 90)
+			(at 171.45 61.9124 90)
 			(effects
 				(font
@@
 		)
 		(property "Footprint" "Diode_SMD:D_SMC"
-			(at 225.425 60.96 0)
+			(at 164.465 60.96 0)
 			(effects
 				(font
@@
 		)
 		(property "Datasheet" "http://www.vishay.com/docs/88946/b120.pdf"
-			(at 229.87 60.96 0)
+			(at 168.91 60.96 0)
 			(effects
 				(font
@@
 		)
 		(property "Description" "20V 1A Schottky Barrier Rectifier Diode, SMA(DO-214AC)"
-			(at 229.87 60.96 0)
+			(at 168.91 60.96 0)
 			(effects
 				(font
@@
 	(symbol
 		(lib_id "Transistor_FET:IRF540N")
-		(at 217.17 59.69 0)
-		(unit 1)
-		(exclude_from_sim no)
-		(in_bom yes)
-		(on_board yes)
-		(dnp no)
-		(fields_autoplaced yes)
+		(at 156.21 59.69 0)
+		(unit 1)
+		(exclude_from_sim no)
+		(in_bom yes)
+		(on_board yes)
+		(dnp no)
 		(property "Reference" "Q2"
-			(at 223.52 58.4199 0)
+			(at 162.56 58.4199 0)
 			(effects
 				(font
@@
 		)
 		(property "Value" "IRF540N"
-			(at 223.52 60.9599 0)
+			(at 162.56 60.9599 0)
 			(effects
 				(font
@@
 		)
 		(property "Footprint" "Package_TO_SOT_THT:TO-220-3_Horizontal_TabDown"
-			(at 222.25 61.595 0)
+			(at 161.29 61.595 0)
 			(effects
 				(font
@@
 		)
 		(property "Datasheet" "http://www.irf.com/product-info/datasheets/data/irf540n.pdf"
-			(at 222.25 63.5 0)
+			(at 161.29 63.5 0)
 			(effects
 				(font
@@
 		)
 		(property "Description" "33A Id, 100V Vds, HEXFET N-Channel MOSFET, TO-220"
-			(at 217.17 59.69 0)
+			(at 156.21 59.69 0)
 			(effects
 				(font
@@
 	(symbol
 		(lib_id "Diode:B120-E3")
-		(at 168.91 60.96 270)
-		(unit 1)
-		(exclude_from_sim no)
-		(in_bom yes)
-		(on_board yes)
-		(dnp no)
-		(fields_autoplaced yes)
+		(at 229.87 60.96 270)
+		(unit 1)
+		(exclude_from_sim no)
+		(in_bom yes)
+		(on_board yes)
+		(dnp no)
 		(property "Reference" "D1"
-			(at 171.45 60.6424 90)
+			(at 232.41 60.6424 90)
 			(effects
 				(font
@@
 		)
 		(property "Value" "B120-E3"
-			(at 171.45 61.9124 90)
+			(at 232.41 61.9124 90)
 			(effects
 				(font
@@
 		)
 		(property "Footprint" "Diode_SMD:D_SMC"
-			(at 164.465 60.96 0)
+			(at 225.425 60.96 0)
 			(effects
 				(font
@@
 		)
 		(property "Datasheet" "http://www.vishay.com/docs/88946/b120.pdf"
-			(at 168.91 60.96 0)
+			(at 229.87 60.96 0)
 			(effects
 				(font
@@
 		)
 		(property "Description" "20V 1A Schottky Barrier Rectifier Diode, SMA(DO-214AC)"
-			(at 168.91 60.96 0)
+			(at 229.87 60.96 0)
 			(effects
 				(font
@@
 	(symbol
 		(lib_id "Transistor_FET:IRF540N")
-		(at 156.21 59.69 0)
+		(at 217.17 59.69 0)
 		(unit 1)
 		(exclude_from_sim no)
@@
 		(fields_autoplaced yes)
 		(property "Reference" "Q1"
-			(at 162.56 58.4199 0)
+			(at 223.52 58.4199 0)
 			(effects
 				(font
@@
 		)
 		(property "Value" "IRF540N"
-			(at 162.56 60.9599 0)
+			(at 223.52 60.9599 0)
 			(effects
 				(font
@@
 		)
 		(property "Footprint" "Package_TO_SOT_THT:TO-220-3_Horizontal_TabDown"
-			(at 161.29 61.595 0)
+			(at 222.25 61.595 0)
 			(effects
 				(font
@@
 		)
 		(property "Datasheet" "http://www.irf.com/product-info/datasheets/data/irf540n.pdf"
-			(at 161.29 63.5 0)
+			(at 222.25 63.5 0)
 			(effects
 				(font
@@
 		)
 		(property "Description" "33A Id, 100V Vds, HEXFET N-Channel MOSFET, TO-220"
-			(at 156.21 59.69 0)
-			(effects
-				(font
+			(at 217.17 59.69 0)
+			(effects
+				(font
