File: arduino_nano_fullbridge_dc_driver/arduino_nano_fullbridge_dc_driver.kicad_sch (KiCad schematic)
At the start: 31 parts, among them J1 Conn_01x06_Pin, J2 Conn_01x02_Pin, J3 Barrel_Jack, J4 Conn_01x02_Pin, Q1 IRF540N, Q2 IRF540N, U1 L7805, U2 PC817, U3 LM358, U4 PC817

Commit message: v1.0.0
Parts:
- removed D5: B120-E3, Diode_SMD:D_SOD-123, symbol Diode:B120-E3
- removed J4: Conn_01x02_Pin, Connector_PinHeader_2.54mm:PinHeader_1x02_P2.54mm_Vertical, symbol Connector:Conn_01x02_Pin
- removed R12: 1k, Resistor_SMD:R_0805_2012Metric, symbol Device:R
- removed R7: 68k, Resistor_SMD:R_0805_2012Metric, symbol Device:R
- removed R8: 39k, Resistor_SMD:R_0805_2012Metric, symbol Device:R
- removed RV2: R_Potentiometer_Trim_US, Potentiometer_THT:Potentiometer_Bourns_3296W_Vertical, symbol Device:R_Potentiometer_Trim_US
- removed unit 1 of U3
- added D1, D3: B120-E3, Diode_SMD:D_SMA, symbol Diode:B120-E3
- added Q1, Q3: IRF9540N, Package_TO_SOT_THT:TO-220-3_Horizontal_TabDown, symbol Transistor_FET:IRF9540N
- added Q5, Q6: BC817, Package_TO_SOT_SMD:SOT-23, symbol Transistor_BJT:BC817
- added R10, R13: 100k, Resistor_SMD:R_0805_2012Metric, symbol Device:R
- added R15, R2: 1k, Resistor_SMD:R_0805_2012Metric, symbol Device:R
- D2: renamed from D1; footprint Diode_SMD:D_SMC -> Diode_SMD:D_SMA
- D4: renamed from D2; footprint Diode_SMD:D_SMC -> Diode_SMD:D_SMA
- J1: value Conn_01x06_Pin -> Conn_01x04_Pin; footprint TerminalBlock_Phoenix:TerminalBlock_Phoenix_MKDS-1,5-6-5.08_1x06_P5.08mm_Horizontal -> TerminalBlock_Phoenix:TerminalBlock_Phoenix_MKDS-1,5-4-5.08_1x04_P5.08mm_Horizontal; symbol Connector:Conn_01x06_Pin -> Connector:Conn_01x04_Pin
- R5, R6: value R -> 560
- renumbered Q1 to Q2, Q2 to Q4
Connections:
- net GND: now also J1.2 (Pin_2), Q5.2 (E), Q6.2 (E); no longer J1.4 (Pin_4)
- net S1: now also R2.1
- net S2: now also R15.1
- net at R14.2, R16.2: now also Q4.1 (G); no longer Q2.1 (G)
- net at R1.2, R9.2: now also Q2.1 (G); no longer Q4.1 (G)
- net A6: no longer names the net of A1.25 (A6)
- removed net L1a: J1.2 (Pin_2), J1.3 (Pin_3), J1.6 (Pin_6)
- net L1b renamed L2
- net L2: now also D3.2 (A), Q3.2 (D)
- net L2b renamed L1
- net L1: now also J1.4 (Pin_4), D1.2 (A), Q1.2 (D); no longer J1.5 (Pin_5)
- new net: Q5.1 (B), R2.2
- new net: Q6.1 (B), R15.2
- new net: Q3.1 (G), Q6.3 (C), R13.1
- new net: Q1.1 (G), Q5.3 (C), R10.1
- new net V+: D1.1 (K), D3.1 (K), J1.3 (Pin_3), Q1.3 (S), Q3.3 (S), R10.2, R13.2
Other:
- moved on the sheet: D2, D4, Q2, Q4
