File: arduino_nano_low_side_dc_driver/arduino_nano_low_side_dc_driver.kicad_sch (KiCad schematic)
At the start: 35 parts, among them J1 Conn_01x04_Pin, J2 Conn_01x02_Pin, J3 Barrel_Jack, Q1 IRF9540N, Q2 IRF540N, Q3 IRF9540N, Q4 IRF540N, Q5 BC817, Q6 BC817, U1 L7805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

Commit message: v1.0.0
Parts:
- removed D1, D3: B120-E3, Diode_SMD:D_SMA, symbol Diode:B120-E3
- removed Q1, Q3: IRF9540N, Package_TO_SOT_THT:TO-220-3_Horizontal_TabDown, symbol Transistor_FET:IRF9540N
- removed Q5, Q6: BC817, Package_TO_SOT_SMD:SOT-23, symbol Transistor_BJT:BC817
- removed R10, R13: 100k, Resistor_SMD:R_0805_2012Metric, symbol Device:R
- removed R15, R2: 1k, Resistor_SMD:R_0805_2012Metric, symbol Device:R
- added D5: B120-E3, Diode_SMD:D_SOD-123, symbol Diode:B120-E3
- added J4: Conn_01x02_Pin, Connector_PinHeader_2.54mm:PinHeader_1x02_P2.54mm_Vertical, symbol Connector:Conn_01x02_Pin
- added R12: 1k, Resistor_SMD:R_0805_2012Metric, symbol Device:R
- added R7: 68k, Resistor_SMD:R_0805_2012Metric, symbol Device:R
- added R8: 39k, Resistor_SMD:R_0805_2012Metric, symbol Device:R
- added RV2: R_Potentiometer_Trim_US, Potentiometer_THT:Potentiometer_Bourns_3296W_Vertical, symbol Device:R_Potentiometer_Trim_US
- added unit 1 of U3
- D1: renamed from D2; footprint Diode_SMD:D_SMA -> Diode_SMD:D_SMC
- D2: renamed from D4; footprint Diode_SMD:D_SMA -> Diode_SMD:D_SMC
- J1: value Conn_01x04_Pin -> Conn_01x06_Pin; footprint TerminalBlock_Phoenix:TerminalBlock_Phoenix_MKDS-1,5-4-5.08_1x04_P5.08mm_Horizontal -> TerminalBlock_Phoenix:TerminalBlock_Phoenix_MKDS-1,5-6-5.08_1x06_P5.08mm_Horizontal; symbol Connector:Conn_01x04_Pin -> Connector:Conn_01x06_Pin
- R5, R6: value R -> 560
- renumbered Q2 to Q1, Q4 to Q2
Connections:
- net 12V: now also D5.2 (A)
- net GND: now also J1.4 (Pin_4), RV2.3; no longer J1.2 (Pin_2)
- net I2: now also R7.2
- net at R14.2, R16.2: now also Q1.1 (G); no longer Q2.1 (G)
- net at R1.2, R9.2: now also Q2.1 (G); no longer Q1.1 (G)
- net A6: now reaches A1.25 (A6)
- net A6: now also U3.1, U3.2 (-)
- net L1 renamed L2b
- net L2b: now also J1.5 (Pin_5); no longer J1.4 (Pin_4)
- net L2 renamed L1b
- net V+ renamed L1a
- net L1a: now also J1.2 (Pin_2), J1.6 (Pin_6), J4.2 (Pin_2)
- new net: R12.1, U3.3 (+)
- new net: D5.1 (K), J4.1 (Pin_1)
- new net: R8.1, RV2.1, RV2.2
- new net: R12.2, R7.1, R8.2
Other:
- moved on the sheet: D1, D2, Q1, Q2
