File: relay_module_12v_optocoupler/relay_module_12v_optocoupler.kicad_pcb (KiCad board)
At the start: 2 copper layers, 26.2 x 67.3 mm, 15 parts, among them J1 Conn_01x02_Pin, J2 Conn_01x03_Pin, K1 Relay_SPDT, Q1 BC337, U1 PC817

Commit message: v1.0.0
Parts:
- moved REF** 0.39 mm to (138.5, 137.4)
- moved REF** 0.38 mm to (159.7, 137.4)
- moved J1 0.08 mm to (154.2, 79.1)
- moved REF** 0.05 mm to (159.7, 75.4)
Other:
- board size 26.2 x 67.3 mm -> 26 x 67 mm
Changed lines of the file:
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@@
 			(outputformat 1)
 			(mirror no)
-			(drillshape 1)
+			(drillshape 0)
 			(scaleselection 1)
-			(outputdirectory "")
+			(outputdirectory "gerbers/")
 		)
 	)
@@
 	(footprint "MountingHole:MountingHole_2.2mm_M2"
 		(layer "F.Cu")
-		(at 159.766 137.795)
+		(at 159.7152 137.414)
 		(descr "Mounting Hole 2.2mm, M2, no annular, generated by kicad-footprint-generator mountinghole.py")
 		(tags "mountinghole M2")
@@
 	(footprint "MountingHole:MountingHole_2.2mm_M2"
 		(layer "F.Cu")
-		(at 159.766 75.4)
+		(at 159.7152 75.4)
 		(descr "Mounting Hole 2.2mm, M2, no annular, generated by kicad-footprint-generator mountinghole.py")
 		(tags "mountinghole M2")
@@
 	(footprint "TerminalBlock_Phoenix:TerminalBlock_Phoenix_MKDS-1,5-3-5.08_1x03_P5.08mm_Horizontal"
 		(layer "F.Cu")
-		(at 154.2746 79.1263 180)
+		(at 154.2 79.1 180)
 		(descr "Terminal Block Phoenix MKDS-1,5-3-5.08, 3 pins, pitch 5.08mm, size 15.2x9.8mm, drill diameter 1.3mm, pad diameter 2.6mm, http://www.farnell.com/datasheets/100425.pdf, script-generated using https://gitlab.com/kicad/libraries/kicad-footprint-generator/-/tree/master/scripts/TerminalBlock_Phoenix")
 		(tags "THT Terminal Block Phoenix MKDS-1,5-3-5.08 pitch 5.08mm size 15.2x9.8mm drill 1.3mm pad 2.6mm")
@@
 		(tags "THT Terminal Block Phoenix MKDS-1,5-3-5.08 pitch 5.08mm size 15.2x9.8mm drill 1.3mm pad 2.6mm")
 		(property "Reference" "J2"
-			(at 5.085 3.048 0)
+			(at 5.08 3.4036 0)
 			(layer "F.SilkS")
 			(effects
@@
 	(footprint "MountingHole:MountingHole_2.2mm_M2"
 		(layer "F.Cu")
-		(at 138.43 137.795)
+		(at 138.5 137.414)
 		(descr "Mounting Hole 2.2mm, M2, no annular, generated by kicad-footprint-generator mountinghole.py")
 		(tags "mountinghole M2")
@@
 		(layer "F.SilkS")
 	)
-	(gr_arc
-		(start 138.2 140.246)
-		(mid 136.644365 139.601635)
-		(end 136 138.046)
+	(gr_line
+		(start 159.8424 139.898)
+		(end 138.2424 139.898)
 		(stroke
 			(width 0.05)
@@
 		(layer "Edge.Cuts")
 	)
-	(gr_line
-		(start 159.996 140.246)
-		(end 138.2 140.246)
+	(gr_arc
+		(start 138.2424 139.898)
+		(mid 136.686765 139.253635)
+		(end 136.0424 137.698)
 		(stroke
 			(width 0.05)
@@
 		(layer "Edge.Cuts")
 	)
-	(gr_line
-		(start 136 138.046)
-		(end 136 75.1)
+	(gr_arc
+		(start 162.0424 137.698)
+		(mid 161.398035 139.253635)
+		(end 159.8424 139.898)
 		(stroke
 			(width 0.05)
@@
 		(layer "Edge.Cuts")
 	)
-	(gr_arc
-		(start 159.996 72.9)
-		(mid 161.551635 73.544365)
-		(end 162.196 75.1)
+	(gr_line
+		(start 136.0424 137.698)
+		(end 136.0424 75.098)
 		(stroke
 			(width 0.05)
@@
 	)
 	(gr_line
-		(start 138.2 72.9)
-		(end 159.996 72.9)
+		(start 138.2424 72.898)
+		(end 159.8424 72.898)
 		(stroke
 			(width 0.05)
@@
 		(layer "Edge.Cuts")
 	)
-	(gr_line
-		(start 162.196 75.1)
-		(end 162.196 138.046)
+	(gr_arc
+		(start 159.8424 72.898)
+		(mid 161.398035 73.542365)
+		(end 162.0424 75.098)
 		(stroke
 			(width 0.05)
@@
 		(layer "Edge.Cuts")
 	)
-	(gr_arc
-		(start 162.196 138.046)
-		(mid 161.551635 139.601635)
-		(end 159.996 140.246)
+	(gr_line
+		(start 162.0424 75.098)
+		(end 162.0424 137.698)
 		(stroke
 			(width 0.05)
@@
 	)
 	(gr_arc
-		(start 136 75.1)
-		(mid 136.644365 73.544365)
-		(end 138.2 72.9)
+		(start 136.0424 75.098)
+		(mid 136.686765 73.542365)
+		(end 138.2424 72.898)
 		(stroke
 			(width 0.05)
@@
 	)
 	(gr_text "DC-"
-		(at 149.1526 73.45 180)
+		(at 149.1526 73.5584 180)
 		(layer "F.SilkS")
 		(effects
@@
 	)
 	(gr_text "IN"
-		(at 154.1526 73.25 180)
+		(at 154.2288 73.5584 180)
 		(layer "F.SilkS")
 		(effects
@@
 	)
 	(gr_text "NO"
-		(at 144.018 139.7 0)
+		(at 143.95 138.95 0)
 		(layer "F.SilkS")
 		(effects
@@
 	)
 	(gr_text "NC"
-		(at 154.25 139.573 0)
+		(at 154.25 138.95 0)
 		(layer "F.SilkS")
 		(effects
@@
 	)
 	(gr_text "COM"
-		(at 149.098 139.7 0)
+		(at 149.098 138.95 0)
 		(layer "F.SilkS")
 		(effects
@@
 	)
 	(gr_text "DC+"
-		(at 144.0526 73.45 180)
+		(at 144.0526 73.5584 180)
 		(layer "F.SilkS")
 		(effects
@@
 		(polygon
 			(pts
-				(xy 136.0152 72.8472) (xy 136.0152 111.0972) (xy 162.306 111.0972) (xy 162.306 72.8472)
+				(xy 136.0576 73) (xy 136.0576 111.0464) (xy 162.0424 110.9492) (xy 162 73)
 			)
 		)

Commit message: v1.0.0
Parts:
- moved J1 0.15 mm to (154.2, 79.2)
Other:
- board text added: "Relay module OPTx1 v1.0"
- board text removed: "Relay module 12V v1.0"
Changed lines of the file:
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@@
 		(tenting front back)
 		(pcbplotparams
-			(layerselection 0x00000000_00000000_55555555_5755f5ff)
+			(layerselection 0x00000000_00000000_55555555_5755557c)
 			(plot_on_all_layers_selection 0x00000000_00000000_00000000_00000000)
 			(disableapertmacros no)
@@
 			(layer "F.Fab")
 		)
-		(fp_text user "K"
-			(at 0 -2.1 0)
-			(layer "F.SilkS")
-			(effects
-				(font
-					(size 1 1)
-					(thickness 0.15)
-				)
-			)
-		)
 		(fp_text user "${REFERENCE}"
 			(at 5.47 0 0)
@@
 	(footprint "TerminalBlock_Phoenix:TerminalBlock_Phoenix_MKDS-1,5-3-5.08_1x03_P5.08mm_Horizontal"
 		(layer "F.Cu")
-		(at 154.2 79.1 180)
+		(at 154.2 79.248 180)
 		(descr "Terminal Block Phoenix MKDS-1,5-3-5.08, 3 pins, pitch 5.08mm, size 15.2x9.8mm, drill diameter 1.3mm, pad diameter 2.6mm, http://www.farnell.com/datasheets/100425.pdf, script-generated using https://gitlab.com/kicad/libraries/kicad-footprint-generator/-/tree/master/scripts/TerminalBlock_Phoenix")
 		(tags "THT Terminal Block Phoenix MKDS-1,5-3-5.08 pitch 5.08mm size 15.2x9.8mm drill 1.3mm pad 2.6mm")
@@
 	(gr_poly
 		(pts
-			(xy 159.492401 81.229001) (xy 159.492401 82.054) (xy 161.4424 82.054) (xy 161.4424 82.804) (xy 161.2924 82.804)
-			(xy 161.2924 82.504) (xy 161.2924 82.354) (xy 159.642401 82.354) (xy 159.642401 82.504) (xy 161.2924 82.504)
-			(xy 161.2924 82.804) (xy 159.492401 82.804) (xy 159.492401 83.629) (xy 159.042401 83.629) (xy 159.042401 81.229001)
+			(xy 159.340001 81.387002) (xy 159.340001 82.212001) (xy 161.29 82.212001) (xy 161.29 82.962001) (xy 161.14 82.962001)
+			(xy 161.14 82.662001) (xy 161.14 82.512001) (xy 159.490001 82.512001) (xy 159.490001 82.662001) (xy 161.14 82.662001)
+			(xy 161.14 82.962001) (xy 159.340001 82.962001) (xy 159.340001 83.787001) (xy 158.890001 83.787001)
+			(xy 158.890001 81.387002)
 		)
 		(stroke
@@
 	(gr_poly
 		(pts
-			(xy 159.942401 85.729) (xy 159.042401 84.979) (xy 159.042401 84.379) (xy 160.242401 85.429) (xy 161.4424 84.379)
-			(xy 161.4424 84.979) (xy 160.542401 85.729) (xy 161.4424 85.729) (xy 161.4424 86.328999) (xy 161.142401 86.328999)
-			(xy 161.142401 86.029) (xy 161.142401 85.879) (xy 159.342401 85.879) (xy 159.342401 86.029) (xy 161.142401 86.029)
-			(xy 161.142401 86.328999) (xy 159.042401 86.328999) (xy 159.042401 85.729)
+			(xy 159.790001 85.887001) (xy 158.890001 85.137001) (xy 158.890001 84.537001) (xy 160.090001 85.587001)
+			(xy 161.29 84.537001) (xy 161.29 85.137001) (xy 160.390001 85.887001) (xy 161.29 85.887001) (xy 161.29 86.487)
+			(xy 160.990001 86.487) (xy 160.990001 86.187001) (xy 160.990001 86.037001) (xy 159.190001 86.037001)
+			(xy 159.190001 86.187001) (xy 160.990001 86.187001) (xy 160.990001 86.487) (xy 158.890001 86.487)
+			(xy 158.890001 85.887001)
 		)
 		(stroke
@@
 	(gr_poly
 		(pts
-			(xy 159.492401 78.229001) (xy 159.492401 79.729001) (xy 159.942401 79.729001) (xy 159.942401 78.229001)
-			(xy 161.4424 78.229001) (xy 161.4424 80.329001) (xy 160.992401 80.329001) (xy 160.992401 78.829001)
-			(xy 160.992401 78.679001) (xy 160.992401 78.529001) (xy 160.542401 78.529001) (xy 160.542401 78.679001)
-			(xy 160.992401 78.679001) (xy 160.992401 78.829001) (xy 160.542401 78.829001) (xy 160.542401 80.329001)
-			(xy 159.942401 80.329001) (xy 159.942401 80.029001) (xy 159.942401 79.879001) (xy 159.492401 79.879001)
-			(xy 159.492401 80.029001) (xy 159.942401 80.029001) (xy 159.942401 80.329001) (xy 159.042401 80.329001)
-			(xy 159.042401 78.229001)
+			(xy 159.340001 78.387002) (xy 159.340001 79.887002) (xy 159.790001 79.887002) (xy 159.790001 78.387002)
+			(xy 161.29 78.387002) (xy 161.29 80.487002) (xy 160.840001 80.487002) (xy 160.840001 78.987002) (xy 160.840001 78.837002)
+			(xy 160.840001 78.687002) (xy 160.390001 78.687002) (xy 160.390001 78.837002) (xy 160.840001 78.837002)
+			(xy 160.840001 78.987002) (xy 160.390001 78.987002) (xy 160.390001 80.487002) (xy 159.790001 80.487002)
+			(xy 159.790001 80.187002) (xy 159.790001 80.037002) (xy 159.340001 80.037002) (xy 159.340001 80.187002)
+			(xy 159.790001 80.187002) (xy 159.790001 80.487002) (xy 158.890001 80.487002) (xy 158.890001 78.387002)
 		)
 		(stroke
@@
 	)
 	(gr_text "DC-"
-		(at 149.1526 73.5584 180)
+		(at 149.1526 73.533 180)
 		(layer "F.SilkS")
 		(effects
 			(font
-				(size 1 1)
+				(size 0.8 1)
 				(thickness 0.15)
 			)
@@
 	)
 	(gr_text "IN"
-		(at 154.2288 73.5584 180)
+		(at 154.2288 73.533 180)
 		(layer "F.SilkS")
 		(effects
 			(font
-				(size 1 1)
+				(size 0.8 1)
 				(thickness 0.15)
 			)
@@
 	)
 	(gr_text "NO"
-		(at 143.95 138.95 0)
+		(at 143.711904 139.192 0)
 		(layer "F.SilkS")
 		(effects
 			(font
-				(size 1 1)
+				(size 0.8 1)
 				(thickness 0.15)
 			)
@@
 	)
 	(gr_text "NC"
-		(at 154.25 138.95 0)
+		(at 154.25 139.192 0)
 		(layer "F.SilkS")
 		(effects
 			(font
-				(size 1 1)
+				(size 0.8 1)
 				(thickness 0.15)
 			)
 		)
 	)
-	(gr_text "Relay module 12V v1.0"
-		(at 161.5948 105.5116 90)
+	(gr_text "Relay module OPTx1 v1.0"
+		(at 161.29 108.331 90)
 		(layer "F.SilkS")
 		(effects
 			(font
-				(size 1 1)
+				(size 0.8 1)
 				(thickness 0.15)
 			)
@@
 	)
 	(gr_text "COM"
-		(at 149.098 138.95 0)
+		(at 149.098 139.192 0)
 		(layer "F.SilkS")
 		(effects
 			(font
-				(size 1 1)
+				(size 0.8 1)
 				(thickness 0.15)
 			)
@@
 	)
 	(gr_text "DC+"
-		(at 144.0526 73.5584 180)
+		(at 144.0526 73.533 180)
 		(layer "F.SilkS")
 		(effects
 			(font
-				(size 1 1)
+				(size 0.8 1)
 				(thickness 0.15)
 			)
@@
 	)
 	(segment
-		(start 154.5135 79.1263)
-		(end 159.9946 84.6074)
+		(start 159.8676 84.9156)
+		(end 159.8676 93.7768)
 		(width 1)
 		(layer "B.Cu")
@@
 	)
 	(segment
-		(start 154.2746 79.1263)
-		(end 154.5135 79.1263)
+		(start 154.2 79.248)
+		(end 159.8676 84.9156)
 		(width 1)
 		(layer "B.Cu")
@@
 	(segment
 		(start 157.8356 95.8088)
-		(end 159.9946 93.6498)
+		(end 159.8676 93.7768)
 		(width 1)
 		(layer "B.Cu")
@@
 	)
 	(segment
-		(start 157.861 106.3965)
-		(end 155.25 109.0075)
+		(start 154.2746 79.1263)
+		(end 154.5135 79.1263)
 		(width 1)
 		(layer "B.Cu")
@@
 	)
 	(segment
-		(start 159.8676 93.7768)
-		(end 159.9946 93.6498)
+		(start 157.861 106.3965)
+		(end 155.25 109.0075)
 		(width 1)
 		(layer "B.Cu")
@@
 	)
 	(segment
-		(start 159.9946 91.4908)
-		(end 159.9946 93.6498)
-		(width 1)
-		(layer "B.Cu")
-		(net 1)
-	)
-	(segment
 		(start 156.8196 93.7768)
 		(end 159.8676 93.7768)
@@
 	)
 	(segment
-		(start 159.9946 84.6074)
-		(end 159.9946 91.4908)
-		(width 1)
-		(layer "B.Cu")
-		(net 1)
-	)
-	(segment
 		(start 157.8356 97.3328)
 		(end 157.8356 95.8088)
@@
 	(segment
 		(start 140.3096 82.9313)
-		(end 144.1146 79.1263)
+		(end 140.3567 82.9313)
+		(width 1)
+		(layer "B.Cu")
+		(net 11)
+	)
+	(segment
+		(start 140.3567 82.9313)
+		(end 144.04 79.248)
 		(width 1)
 		(layer "B.Cu")
@@
 		(polygon
 			(pts
-				(xy 136.0576 73) (xy 136.0576 111.0464) (xy 162.0424 110.9492) (xy 162 73)
+				(xy 136.0576 73) (xy 136.017406 110.61819) (xy 162.041976 110.569392) (xy 162 73)
 			)
 		)
@@
 		(polygon
 			(pts
-				(xy 144.945839 111) (xy 144.945839 106.5) (xy 146.945839 104.5) (xy 151.945839 104.5) (xy 153.445839 106)
-				(xy 153.445839 111)
+				(xy 145.161 110.613193) (xy 145.161 106.045) (xy 147.066 104.521) (xy 151.531551 104.494193) (xy 153.407 105.994193)
+				(xy 153.407 110.613193)
 			)
 		)

Commit message: v1.0.0
Routing:
- net Net-(R2-Pad2): track 12.2 -> 11.7 mm
Changed lines of the file:
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@@
 		(tags "THT DIP DIL PDIP 2.54mm 7.62mm 300mil")
 		(property "Reference" "U1"
-			(at 3.81 1.275 90)
+			(at 3.81 1.275 180)
 			(layer "F.SilkS")
 			(effects
@@
 		(start 143.2306 132.5626)
 		(end 144.018 133.35)
-		(width 3.5)
+		(width 4.2)
 		(layer "B.Cu")
 		(net 2)
@@
 		(start 143.2306 121.3866)
 		(end 143.2306 132.5626)
-		(width 3.5)
+		(width 4.2)
 		(layer "B.Cu")
 		(net 2)
 	)
 	(segment
-		(start 149.2306 107.1866)
-		(end 149.2306 133.2174)
-		(width 3.5)
+		(start 149.098 107.3192)
+		(end 149.2306 107.1866)
+		(width 4.2)
 		(layer "B.Cu")
 		(net 3)
 	)
 	(segment
-		(start 149.2306 133.2174)
-		(end 149.098 133.35)
-		(width 3.5)
+		(start 149.098 133.35)
+		(end 149.098 107.3192)
+		(width 4.2)
 		(layer "B.Cu")
 		(net 3)
@@
 		(start 155.2306 132.2974)
 		(end 154.178 133.35)
-		(width 3.5)
+		(width 4.2)
 		(layer "B.Cu")
 		(net 4)
@@
 		(start 155.2306 121.3866)
 		(end 155.2306 132.2974)
-		(width 3.5)
+		(width 4.2)
 		(layer "B.Cu")
 		(net 4)
@@
 	(segment
 		(start 150.3172 86.6648)
-		(end 153.1366 89.4842)
+		(end 152.4508 88.7984)
 		(width 1)
 		(layer "B.Cu")
@@
 	)
 	(segment
+		(start 155.5242 88.7984)
+		(end 156.8196 87.503)
+		(width 1)
+		(layer "B.Cu")
+		(net 9)
+	)
+	(segment
 		(start 156.8196 87.503)
-		(end 154.8384 89.4842)
-		(width 1)
-		(layer "B.Cu")
-		(net 9)
-	)
-	(segment
-		(start 156.8196 86.1568)
-		(end 156.8196 87.503)
-		(width 1)
-		(layer "B.Cu")
-		(net 9)
-	)
-	(segment
-		(start 153.1366 89.4842)
-		(end 154.8384 89.4842)
+		(end 156.8196 86.1568)
 		(width 1)
 		(layer "B.Cu")
@@
 		(start 147.9296 86.6648)
 		(end 150.3172 86.6648)
+		(width 1)
+		(layer "B.Cu")
+		(net 9)
+	)
+	(segment
+		(start 152.4508 88.7984)
+		(end 155.5242 88.7984)
 		(width 1)
 		(layer "B.Cu")
@@
 		(layer "B.Cu")
 		(hatch edge 0.5)
-		(connect_pads
+		(connect_pads yes
 			(clearance 0.5)
 		)
@@
 		(polygon
 			(pts
-				(xy 136.0576 73) (xy 136.017406 110.61819) (xy 162.041976 110.569392) (xy 162 73)
-			)
-		)
+				(xy 136.0424 72.898) (xy 136.0424 110.6424) (xy 162.052 110.6424) (xy 162.052 72.898)
+			)
+		)
