File: relay_module_12v_optocoupler/relay_module_12v_optocoupler.kicad_sch (KiCad schematic)
At the start: 11 parts, among them J1 Conn_01x02_Pin, J2 Conn_01x03_Pin, K1 Relay_SPDT, Q1 BC337, U1 PC817

Commit message: v1.0.0
Parts:
- D2: value LED -> LED 3mm
- R3: value R -> 10k
- R4: value R -> 100k
Changed lines of the file:
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@@
 			)
 		)
-		(property "Value" "R"
+		(property "Value" "10k"
 			(at 149.86 120.65 90)
 			(effects
@@
 			)
 		)
-		(property "Value" "R"
+		(property "Value" "100k"
 			(at 158.75 138.4299 0)
 			(effects
@@
 			)
 		)
-		(property "Value" "LED"
+		(property "Value" "LED 3mm"
 			(at 187.198 106.68 90)
 			(effects
