File: relay_module_12v_optocoupler_smt/relay_module_12v_optocoupler_smt.kicad_pcb (KiCad board)
At the start: 2 copper layers, 27.2 x 59.1 mm, 15 parts, among them J1 Conn_01x02_Pin, J2 Conn_01x03_Pin, K1 Relay_SPDT, Q2 BC817, U1 PC817

Commit message: v1.0.0
Changed lines of the file:
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@@
 			(outputformat 1)
 			(mirror no)
-			(drillshape 1)
+			(drillshape 0)
 			(scaleselection 1)
-			(outputdirectory "")
+			(outputdirectory "gerbers/")
 		)
 	)
@@
 	(gr_poly
 		(pts
-			(xy 159.8 86.1375) (xy 160.25 86.5125) (xy 160.25 86.8125) (xy 159.65 86.2875) (xy 159.05 86.8125)
-			(xy 159.05 86.5125) (xy 159.5 86.1375) (xy 159.05 86.1375) (xy 159.05 85.8375) (xy 159.2 85.8375)
-			(xy 159.2 85.9875) (xy 159.2 86.0625) (xy 160.1 86.0625) (xy 160.1 85.9875) (xy 159.2 85.9875) (xy 159.2 85.8375)
-			(xy 160.25 85.8375) (xy 160.25 86.1375)
+			(xy 159.7732 86.064401) (xy 160.2232 86.439401) (xy 160.2232 86.739401) (xy 159.6232 86.214401) (xy 159.0232 86.739401)
+			(xy 159.0232 86.439401) (xy 159.4732 86.064401) (xy 159.0232 86.064401) (xy 159.0232 85.764401) (xy 159.1732 85.764401)
+			(xy 159.1732 85.914401) (xy 159.1732 85.989401) (xy 160.0732 85.989401) (xy 160.0732 85.914401) (xy 159.1732 85.914401)
+			(xy 159.1732 85.764401) (xy 160.2232 85.764401) (xy 160.2232 86.064401)
 		)
 		(stroke
@@
 	(gr_poly
 		(pts
-			(xy 160.025 89.887499) (xy 160.025 89.1375) (xy 159.8 89.1375) (xy 159.8 89.887499) (xy 159.05 89.887499)
-			(xy 159.05 88.8375) (xy 159.275 88.8375) (xy 159.275 89.5875) (xy 159.275 89.6625) (xy 159.275 89.737499)
-			(xy 159.5 89.737499) (xy 159.5 89.6625) (xy 159.275 89.6625) (xy 159.275 89.5875) (xy 159.5 89.5875)
-			(xy 159.5 88.8375) (xy 159.8 88.8375) (xy 159.8 88.9875) (xy 159.8 89.0625) (xy 160.025 89.0625)
-			(xy 160.025 88.9875) (xy 159.8 88.9875) (xy 159.8 88.8375) (xy 160.25 88.8375) (xy 160.25 89.887499)
+			(xy 159.9982 89.8144) (xy 159.9982 89.064401) (xy 159.7732 89.064401) (xy 159.7732 89.8144) (xy 159.0232 89.8144)
+			(xy 159.0232 88.764401) (xy 159.2482 88.764401) (xy 159.2482 89.514401) (xy 159.2482 89.589401) (xy 159.2482 89.6644)
+			(xy 159.4732 89.6644) (xy 159.4732 89.589401) (xy 159.2482 89.589401) (xy 159.2482 89.514401) (xy 159.4732 89.514401)
+			(xy 159.4732 88.764401) (xy 159.7732 88.764401) (xy 159.7732 88.914401) (xy 159.7732 88.989401) (xy 159.9982 88.989401)
+			(xy 159.9982 88.914401) (xy 159.7732 88.914401) (xy 159.7732 88.764401) (xy 160.2232 88.764401) (xy 160.2232 89.8144)
 		)
 		(stroke
@@
 	(gr_poly
 		(pts
-			(xy 160.025 88.3875) (xy 160.025 87.975) (xy 159.05 87.975) (xy 159.05 87.6) (xy 159.125 87.6) (xy 159.125 87.75)
-			(xy 159.125 87.825) (xy 159.95 87.825) (xy 159.95 87.75) (xy 159.125 87.75) (xy 159.125 87.6) (xy 160.025 87.6)
-			(xy 160.025 87.1875) (xy 160.25 87.1875) (xy 160.25 88.3875)
+			(xy 159.9982 88.314401) (xy 159.9982 87.901901) (xy 159.0232 87.901901) (xy 159.0232 87.526901) (xy 159.0982 87.526901)
+			(xy 159.0982 87.676901) (xy 159.0982 87.751901) (xy 159.9232 87.751901) (xy 159.9232 87.676901) (xy 159.0982 87.676901)
+			(xy 159.0982 87.526901) (xy 159.9982 87.526901) (xy 159.9982 87.114401) (xy 160.2232 87.114401) (xy 160.2232 88.314401)
 		)
 		(stroke
@@
 	)
 	(segment
-		(start 143.144 119.946)
-		(end 143.144 131.349)
-		(width 3.5)
+		(start 143.144 131.349)
+		(end 144.005 132.21)
+		(width 4.2)
 		(layer "B.Cu")
 		(net 2)
 	)
 	(segment
-		(start 143.144 131.349)
-		(end 144.005 132.21)
-		(width 3.5)
+		(start 143.144 119.946)
+		(end 143.144 131.349)
+		(width 4.2)
 		(layer "B.Cu")
 		(net 2)
 	)
 	(segment
-		(start 149.144 132.151)
-		(end 149.085 132.21)
-		(width 3.5)
+		(start 149.085 132.21)
+		(end 149.085 105.805)
+		(width 4.2)
 		(layer "B.Cu")
 		(net 3)
 	)
 	(segment
-		(start 149.144 105.746)
-		(end 149.144 132.151)
-		(width 3.5)
+		(start 149.085 105.805)
+		(end 149.144 105.746)
+		(width 4.2)
 		(layer "B.Cu")
 		(net 3)
@@
 		(start 155.144 131.231)
 		(end 154.165 132.21)
-		(width 3.5)
+		(width 4.2)
 		(layer "B.Cu")
 		(net 4)
@@
 		(start 155.144 119.946)
 		(end 155.144 131.231)
-		(width 3.5)
+		(width 4.2)
 		(layer "B.Cu")
 		(net 4)
@@
 		(polygon
 			(pts
-				(xy 136 80.5) (xy 162.25 80.5) (xy 162.25 108.75) (xy 136 108.75)
+				(xy 136 80.5) (xy 162.25 80.5) (xy 162.25 108.712) (xy 136 108.712)
 			)
 		)
@@
 		(layer "B.Cu")
 		(hatch edge 0.5)
-		(connect_pads
-			(clearance 0.7)
+		(connect_pads yes
+			(clearance 0.75)
 		)
 		(min_thickness 0.25)
@@
 		(polygon
 			(pts
-				(xy 136 80.342001) (xy 136 108.75) (xy 162.25 108.724052) (xy 162.25 80.342001)
+				(xy 136 80.342001) (xy 136 108.712) (xy 162.2552 108.712) (xy 162.25 80.342001)
 			)
 		)
