File: relay_module_12v_optocoupler_smt/relay_module_12v_optocoupler_smt.kicad_sch (KiCad schematic)
At the start: 11 parts, among them J1 Conn_01x02_Pin, J2 Conn_01x03_Pin, K1 Relay_SPDT, Q2 BC817, U1 PC817

Commit message: v1.0.0
Parts:
- R3: value R -> 10k
- R4: value R -> 100k
Changed lines of the file:
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@@
 			)
 		)
-		(property "Value" "R"
+		(property "Value" "10k"
 			(at 151.13 111.76 90)
 			(effects
@@
 			)
 		)
-		(property "Value" "R"
+		(property "Value" "100k"
 			(at 160.02 129.5399 0)
 			(effects
