File: relay_module_24v_4/relay_module_24v_4.kicad_pcb (KiCad board)
At the start: 2 copper layers, 77.1 x 67.6 mm, 22 parts, among them J1 Conn_01x12_Pin, J4 Conn_01x05_Pin, K1 Relay_SPDT, K2 Relay_SPDT, K3 Relay_SPDT, K4 Relay_SPDT

Commit message: v1.0.0
Changed lines of the file:
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@@
 			(outputformat 1)
 			(mirror no)
-			(drillshape 1)
+			(drillshape 0)
 			(scaleselection 1)
-			(outputdirectory "")
+			(outputdirectory "gerbers/")
 		)
 	)
@@
 		(tags "THT Terminal Block Phoenix MKDS-1,5-5-5.08 pitch 5.08mm size 25.4x9.8mm drill 1.3mm pad 2.6mm")
 		(property "Reference" "J4"
-			(at 24.262 -0.051 90)
+			(at 24.262 -0.051 180)
 			(layer "F.SilkS")
 			(effects
@@
 		(start 104.216573 125.857573)
 		(end 98.820573 120.461573)
-		(width 3.5)
+		(width 4)
 		(layer "B.Cu")
 		(net 10)
@@
 		(start 98.820573 120.461573)
 		(end 98.820573 109.577573)
-		(width 3.5)
+		(width 4)
 		(layer "B.Cu")
 		(net 10)
@@
 		(start 152.505573 109.577573)
 		(end 152.505573 113.824573)
-		(width 3.5)
+		(width 4)
 		(layer "B.Cu")
 		(net 11)
@@
 		(start 152.505573 113.824573)
 		(end 149.936573 116.393573)
-		(width 3.5)
+		(width 4)
 		(layer "B.Cu")
 		(net 11)
@@
 		(start 149.936573 125.857573)
 		(end 149.936573 116.393573)
-		(width 3.5)
+		(width 4)
 		(layer "B.Cu")
 		(net 11)
@@
 		(start 116.715573 114.008573)
 		(end 119.456573 116.749573)
-		(width 3.5)
+		(width 4)
 		(layer "B.Cu")
 		(net 12)
@@
 		(start 119.456573 116.749573)
 		(end 119.456573 125.857573)
-		(width 3.5)
+		(width 4)
 		(layer "B.Cu")
 		(net 12)
@@
 		(start 116.715573 109.577573)
 		(end 116.715573 114.008573)
-		(width 3.5)
+		(width 4)
 		(layer "B.Cu")
 		(net 12)
 	)
 	(segment
-		(start 139.776573 125.857573)
-		(end 139.776573 96.211573)
-		(width 3.5)
+		(start 139.776573 96.211573)
+		(end 140.610573 95.377573)
+		(width 4)
 		(layer "B.Cu")
 		(net 13)
 	)
 	(segment
-		(start 139.776573 96.211573)
-		(end 140.610573 95.377573)
-		(width 3.5)
+		(start 139.776573 125.857573)
+		(end 139.776573 96.211573)
+		(width 4)
 		(layer "B.Cu")
 		(net 13)
@@
 		(start 129.616573 125.857573)
 		(end 129.616573 110.478573)
-		(width 3.5)
+		(width 4)
 		(layer "B.Cu")
 		(net 14)
@@
 		(start 129.616573 110.478573)
 		(end 128.715573 109.577573)
-		(width 3.5)
+		(width 4)
 		(layer "B.Cu")
 		(net 14)
@@
 		(start 144.856573 125.857573)
 		(end 144.856573 111.331573)
-		(width 3.5)
+		(width 4)
 		(layer "B.Cu")
 		(net 15)
@@
 		(start 144.856573 111.331573)
 		(end 146.610573 109.577573)
-		(width 3.5)
+		(width 4)
 		(layer "B.Cu")
 		(net 15)
@@
 		(start 134.696573 125.857573)
 		(end 134.696573 109.663573)
-		(width 3.5)
+		(width 4)
 		(layer "B.Cu")
 		(net 16)
 	)
 	(segment
-		(start 155.016573 125.857573)
-		(end 155.016573 120.313573)
-		(width 3.5)
-		(layer "B.Cu")
-		(net 17)
-	)
-	(segment
-		(start 158.505573 116.824573)
+		(start 158.505573 117.490827)
 		(end 158.505573 95.377573)
-		(width 3.5)
+		(width 4)
 		(layer "B.Cu")
 		(net 17)
 	)
 	(segment
-		(start 155.016573 120.313573)
-		(end 158.505573 116.824573)
-		(width 3.5)
+		(start 155.016573 120.979827)
+		(end 158.505573 117.490827)
+		(width 4)
 		(layer "B.Cu")
 		(net 17)
 	)
 	(segment
-		(start 109.296573 125.857573)
-		(end 109.296573 122.989573)
-		(width 3.5)
+		(start 155.016573 125.857573)
+		(end 155.016573 120.979827)
+		(width 4)
 		(layer "B.Cu")
-		(net 18)
+		(net 17)
 	)
 	(segment
-		(start 109.296573 122.989573)
-		(end 104.818573 118.511573)
-		(width 3.5)
+		(start 109.296573 123.520573)
+		(end 104.820573 119.044573)
+		(width 4)
 		(layer "B.Cu")
 		(net 18)
 	)
 	(segment
-		(start 104.818573 118.511573)
-		(end 104.820573 118.509573)
-		(width 3.5)
+		(start 109.296573 125.857573)
+		(end 109.296573 123.520573)
+		(width 4)
 		(layer "B.Cu")
 		(net 18)
 	)
 	(segment
-		(start 104.820573 118.509573)
+		(start 104.820573 119.044573)
 		(end 104.820573 95.377573)
-		(width 3.5)
+		(width 4)
 		(layer "B.Cu")
 		(net 18)
@@
 		(start 114.418573 120.711573)
 		(end 110.820573 117.113573)
-		(width 3.5)
+		(width 4)
 		(layer "B.Cu")
 		(net 19)
@@
 		(start 110.820573 117.113573)
 		(end 110.820573 109.577573)
-		(width 3.5)
+		(width 4)
 		(layer "B.Cu")
 		(net 19)
@@
 		(start 114.376573 125.857573)
 		(end 114.376573 120.753573)
-		(width 3.5)
-		(layer "B.Cu")
-		(net 19)
-	)
-	(segment
-		(start 114.376573 120.753573)
-		(end 114.418573 120.711573)
-		(width 3.5)
+		(width 4)
 		(layer "B.Cu")
 		(net 19)
@@
 		(start 164.505573 121.448573)
 		(end 164.505573 109.577573)
-		(width 3.5)
+		(width 4)
 		(layer "B.Cu")
 		(net 20)
@@
 		(start 160.096573 125.857573)
 		(end 164.505573 121.448573)
-		(width 3.5)
+		(width 4)
 		(layer "B.Cu")
 		(net 20)
 	)
 	(segment
-		(start 122.715573 112.572573)
-		(end 122.715573 95.377573)
-		(width 3.5)
+		(start 124.536573 125.857573)
+		(end 124.536573 113.106573)
+		(width 4)
 		(layer "B.Cu")
 		(net 21)
 	)
 	(segment
-		(start 124.536573 114.393573)
-		(end 124.536573 125.857573)
-		(width 3.5)
+		(start 122.715573 111.285573)
+		(end 122.715573 95.377573)
+		(width 4)
 		(layer "B.Cu")
 		(net 21)
 	)
 	(segment
-		(start 124.536573 114.393573)
-		(end 122.715573 112.572573)
-		(width 3.5)
+		(start 124.536573 113.106573)
+		(end 122.715573 111.285573)
+		(width 4)
 		(layer "B.Cu")
 		(net 21)
@@
 		(layer "B.Cu")
 		(hatch edge 0.5)
-		(connect_pads
-			(clearance 0.5)
+		(connect_pads yes
+			(clearance 0.75)
 		)
 		(min_thickness 0.25)
@@
 		(polygon
 			(pts
-				(xy 93.738573 64.611573) (xy 93.805995 90.587249) (xy 170.764573 90.870144) (xy 170.764573 64.643573)
+				(xy 93.738573 64.611573) (xy 93.8276 90.932) (xy 170.764573 90.932) (xy 170.764573 64.643573)
 			)
 		)
